File: pcb/OTM-02.sch (KiCad schematic (older format))
At the start: 90 parts, among them J1 USB_MICRO_AB, J2 FH19SC-10S-0.5SH(05), J3 AHCL, M1 304-103, P1 DBG_VCC, P2 DBG_SWDIO, P3 DBG_GND, P4 DBG_SWCLK, P5 DBG_SWO, P7 DBG_RESETn, Q1 FK6K02010L, Q2 MTM761110LBF, Q3 PDTC114EE, Q4 FK6K02010L, SW1 KMS221GPLFS, SW2 KMS221GPLFS, SW3 KMS221GPLFS, SW4 KMS221GPLFS, SW5 KMS221GPLFS, U1 EFM32LG330F256, U2 MAX17043G+U, U3 MCP73831T-2ACI/MC, U4 TPS78230DRVT, U5 TPS78230DRVT, X1 ABS06-32.768KHZ-9-1-T, X2 ABM11-48.000MHZ-B7G-T

Commit message: Rev.M - Accelerometer (ADXL362) added to PCB
This commit reflects the OTM-02-Rev.M PCB's as manufactured in Feb 2013.

Some GPIO rerouting was required to add the ADXL362.

As of commit date, the Memory LCD display, USB recharge circuit, five (5)
switches and vibratory motor all appear to be functioning as intended. The LED
GPIO also functions, however no LED has yet been connected. PWM on the
LED GPIO *may* require implementing to prevent damage to the LED and/or
GPIO.

The following circuits (i.e. software communication) are yet to be tested:
Accelerometer, Li-Po fuel gauge.
Parts:
- removed C25: 1U, symbol C
- removed Q4: FK6K02010L, WSMini6-F1-B, symbol MOS_N_6LEAD
- removed R13: 150R, symbol R
- removed R18: 20R, symbol R
- removed R19: 1K, symbol R
- removed R4: 100K, symbol R
- removed R9: 4K7, symbol R
- removed U2: MAX17043G+U, symbol MAX17043G+U
- added C23, C24: 100N, symbol C
- added R15: 10R, symbol R
- added U2: ADXL362, symbol ADXL362
- added U6: MAX17048G+, symbol MAX17048G+
- renumbered C21 to C20, C22 to C21, C23 to C22, C24 to C25, C20 to C33, C33 to C34, R15 to R10, R16 to R11, R7 to R12, R8 to R13, R20 to R14, R21 to R16, R10 to R4, R11 to R7, R12 to R8, R14 to R9
Connections:
- net labels added: ACCEL_INT, ACCEL_MISO, ACCEL_MOSI, ACCEL_SCLK, ACCEL_~CS~
- net labels removed: FG_BATT_ALRT, RTC_CLKOE, RTC_CLKOUT, RTC_INT, RTC_MISO, RTC_MOSI, RTC_SCK, RTC_SSEL
- wire segments 334 -> 325
- no-connect marks 37 -> 29
Other:
- note added: "------>>\nNOTES\n------>>"
- note added: "Accelerometer"
- note added: "Drive LED using\n<GPIO_Px_CTRL DRIVEMODE = STANDARD> and PWM.\nValue of R to be confirmed.\nMax current for ASMT-CW00 is 10mA. VF varies\nfrom 2.55V (min) - 3.15V (max).\nAt 3V VMCU + Standard drive level, with draw of 10mA,\nGPIO voltage drops to approx 2.7V.\nThis should be sufficient to prevent LED drawing"
- note added: "RES PINS - May be connected to ground or left unconnected.\nNC PINS - Not internally connected."
- note added: "• THIS IS A WORK IN PROGRESS,\nCONSIDER IT A STARTING POINT.\nLatest version is available at:\ngithub.com/hairykiwi/OTM-02\n\n• U1 Pin/function locations to be optimised\naccording to PCB layout requirements.\n\n• All XX_PUSHER MCU inputs coincide\nwith Low Energy Sense (LES)\ninputs for potential implementation of\ncapacitive touch button UI."
- note removed: "-----------------------------\nNOTES\n-----------------------------\n• U1 Pin/function locations to be optimised\naccording to PCB layout requirements.\n\n• Extra juntions shown throughout circuit\nare remnants of Test Points which could be\nreinstated, space permitting.\n\n• All XX_PUSHER MCU inputs coincide\nwith Low Energy Sense (LES)\ninputs for potential implementation of\ncapacitive touch b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"
- note removed: "NOTE: RTC (1024 Hz) is Option B"
- note removed: "NOTE: THIS IS A WORK IN PROGRESS.\nFOR DERIVATIVES, CONSIDER IT A STARTING POINT.\nLatest version will be made available either at:\ngithub.com/hairykiwi/OTM-02"
- note removed: "RTC"
- note removed: "RV-3049 - Configure for 1024Hz CLKOUT - EXPERIMENTAL\n\nRemoved for PCB DRC\nLast included in Rev.D saved 2012-11-29 15:49 UTC"
- note removed: "USART1_#1 - pins 28 - 31:\nProbably the best physical\nlocation for connecting a SPI\nenabled accelerometer."
- note removed: "Zero ohm links R12/R13\nremoved at RevH.\nCaution: Original firmware\nconfigured for SW_VCOM.\n\nHW_VCOM:\nR12 Installed,\nR13 Omitted.\n\nSW_VCOM:\nR27 Installed,\nR19 Omitted."
- moved on the sheet: C13, C20, C21, C27, C33, D1, D2, D3, J2, LED1, M1, PAD1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

Commit message: Retrospective commit message correction + housekeeping + minor updates.
The previous commit message omitted some of the major changes
between Rev.L and Rev.M.
The major changes as of the previous commit (initial commit of rev.M) were:
- Accelerometer added (ADXL362).
- Battery 'Fuel Gauge' IC (MAX17043G+U) updated to smaller (MAX17048G+).
- Backlight LED switched directly by EFM32, (i.e. MOSFET switch removed).

Changes introduced as of *this* commit:
- Debug Interface 'P7' relabelled 'P6', to reflect actual total pin count.
- Piezoelectric diaphragm (PED) connections (pads) labelled 'PADx',
  relabelled 'SPx' to better reflect the Spring Pin component fitted.
- PED SP module (PCB footprint) - outline now depicted in 'Dwgs.User' layer.
- Component 'PIEZO_DIAPHRAGM-DUMMY' added to enable inclusion of the PED
  in the Bill of Materials (BOM), without generating a physical board-mounted
  component in Pcbnew.
- Schematic layout - minor tidying.
- OTM-02_bom-colour_coded.pdf - added. A google docs based, colour-coded BOM:
  https://docs.google.com/spreadsheet/ccc?key=0AiBBK0ta6UF0dHBZZUZtNGNDcU9SalJwMnNUR1ctb2c&usp=sharing
- OTM-02_assy_drawing-colour_coded.pdf added. (Begins life as SVG plot in Pcbnew,
  further edited and coloured in Inkscape.
- OTM-02_assy_drawing.pdf - removed. (Due poor quality.)
- OTM-02.dcm documentation file added.

NB: All changes as of this commit are compatible with the first batch of
Rev.M PCBs manufactured.
Parts:
- added X3: 7BB-20-3, symbol PIEZO_DIAPHRAGM-DUMMY
- C16, C18, C22, C31: Voltage (none) -> 10VDC
- J3: value AHCL -> ACHLR-02V-S; Alt Value (none) -> ACHR-02V-S
- SP1: renamed from PAD1; value PIEZO_PAD1 -> 0910-1-57-20-75-14-11-0
- SP2: renamed from PAD2; value PIEZO_PAD2 -> 0910-1-57-20-75-14-11-0
- X1: Value_Alt (none) -> ABS06-32.768KHZ-9-1-T
- renumbered P7 to P6
Connections:
- wire segments 325 -> 322
- no-connect marks 29 -> 28
Other:
- note added: "- For reference designs, recommendations and app notes\nsee: http://bit.ly/Mey1VI and\nhttp://www.precisionmicrodrives.com/application-notes-technical-guides\n- Consider using X2Y 6R3X14W104MV4T for bypass\nfiltering (Farnell code: 1886132)\nDetails here: http://johansondielectrics.com/x2y-products.html"
- note added: "------------>>\nGENERAL NOTES\n------------>>"
- note added: "304-103 (Permanent Magnet Motor):\nPerf Characteristics: For Vdd = 3.0V, I = 73 mA\nPWM Calcs:\nL = 600uH\nFor C = 100nF - F(r) = 20.5kHz\nFor C = 100pF - F(r) = 650kHz\n\nNOTE: If M1 substituted with brushless motor,\nPWM is NOT permitted."
- note added: "Battery:\nLi-Po 3.7V 150mAh\nP/N: CS-IPSF5SL\n15*24*2.5mm"
- note added: "CHANGES: Accelerometer added. Fuel Gauge IC updated to latest (smaller) model. Backlight LED now switched directly by MCU."
- note added: "Drive LED using <GPIO_Px_CTRL DRIVEMODE =\nSTANDARD> + PWM.\n- Value of R to be confirmed.\n- Max current for ASMT-CW00 is 10mA.\n- VF varies from 2.55V (min) - 3.15V (max).\n- At 3V VMCU + Standard drive level,\nwith draw of 10mA, GPIO voltage drops\nto approx 2.7V. As a result, LED should \nnot be able to draw excess current."
- note added: "MEMORY LCD NOTES\n--------------------------\nEXTMODE:\nWhen <H>, EXTCOMIN signal is enable.\nWhen <L> ,serial input flag is enable.\n\nC12 &C13 100N MINIMUM -\nMay be 1U for convenience."
- note added: "Major experimenting required with Hesaglas (0.3 - 0.5mm cast\nacrylic) + laser engraving to construct a planar lightguide as\ndescribed by Idé et al.\n"
- note added: "R10\n10K = approx. 100mA charge current\n5K = approx. 200mA charge current"
- note added: "Replace ACHLR-02V-S:\nheight:1.2 mm,\nwith readily available ACHR-02V-S:\nheight: 1.4 mm"
- note added: "SP1 & SP2 P/N:"
- note added: "SP1 & SP2:\nMILL-MAX 0910-1\nSpring-Loaded Pin - SMD\nInitial Height: 4.5 mm - Stroke: 1.4 mm\n\nAlternative:\n0930 Spring-Loaded Pin - TH SOLDERTAIL\nInitial Height: 4.4 mm - Stroke: 1.4 mm"
- note added: "X3 typically mounted in case-back\nand connected via SP1 & SP2 using\nspring-loaded contacts.\nP/N Details:\n7BB-20-3: 20 mm dia, leadless\n7BB-20-6L0: 20 mm dia, with\n32AWG x 50 mm flying leads."
- note added: "• THIS IS A WORK IN PROGRESS, CONSIDER IT A STARTING POINT.\n\n• Latest version is available at: github.com/hairykiwi/OTM-02\n\n• U1 Pin/function locations to be optimised according to PCB layout requirements.\n\n• All XX_PUSHER MCU inputs coincide with Low Energy Sense (LES)\ninputs for ease of implementing capacitive touch button UI in alternate PCB layout."
- note removed: "- For reference designs, recommendations and app notes\nsee: http://bit.ly/Mey1VI and\nhttp://www.precisionmicrodrives.com/application-notes-technical-guides\n\n- Consider using X2Y 6R3X14W104MV4T for bypass\nfiltering (Farnell code: 1886132)\nDetails here: http://johansondielectrics.com/x2y-products.html"
- note removed: "------>>\nNOTES\n------>>"
- note removed: "Battery:\nLi-Po\nCS-IPSF5SL\n3V7 150mAh\n15*24*2.5mm"
- note removed: "C12 &C13 100N MINIMUM -\nMay be 1U for convenience."
- note removed: "CHANGES: Krenv1.3 used to realign component numbering (Except P1-P5 & P7) with module XY PCB location."
- note removed: "Drive LED using\n<GPIO_Px_CTRL DRIVEMODE = STANDARD> and PWM.\nValue of R to be confirmed.\nMax current for ASMT-CW00 is 10mA. VF varies\nfrom 2.55V (min) - 3.15V (max).\nAt 3V VMCU + Standard drive level, with draw of 10mA,\nGPIO voltage drops to approx 2.7V.\nThis should be sufficient to prevent LED drawing"
- note removed: "EXTMODE:\nWhen <H>, EXTCOMIN signal is enable.\nWhen <L> ,serial input flag is enable."
- note removed: "Major experimenting required with Hesaglas (0.3 - 0.5mm cast\nacrylic) + laser engraving to construct a planar lightguide\nas described by Idé et al:"
- note removed: "NOTE: LFXO (32,768kHz) is Option A"
- note removed: "NOTE: No PWM permitted with brushless motors."
- note removed: "PWM of 304-103 (Permanent Magnet Motor):\nL = 600uH\nFor C = 100nF - F(r) = 20.5kHz\nFor C = 100pF - F(r) = 650kHz"
- note removed: "Perf Characteristics: For Vdd = 3.0V, I = 73 mA"
- note removed: "Piezoelectric Diaphragm (X3) P/N: 7BB-20-3"
- note removed: "R1\n10K = approx. 100mA charge current\n5K = approx. 200mA charge current"
- note removed: "• THIS IS A WORK IN PROGRESS,\nCONSIDER IT A STARTING POINT.\nLatest version is available at:\ngithub.com/hairykiwi/OTM-02\n\n• U1 Pin/function locations to be optimised\naccording to PCB layout requirements.\n\n• All XX_PUSHER MCU inputs coincide\nwith Low Energy Sense (LES)\ninputs for potential implementation of\ncapacitive touch button UI."
- moved on the sheet: C13, C20, C21, C22, C23, C24, C25, C27, C28, C30, C33, D1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
